File: PCB/BM62-Audio/_autosave-BM62-Audio.kicad_sch (KiCad schematic)
At the start: 3 parts, among them J1 AudioJack3, J2 USB_C_Receptacle_USB2.0

Commit message: ✨ KiCADファイル作りました
Parts:
- J2: footprint (none) -> Connector_USB:USB_C_Receptacle_Palconn_UTC16-G
Changed lines of the file:
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@@
       (effects (font (size 1.27 1.27)))
     )
-    (property "Footprint" "" (at 162.56 67.31 0)
+    (property "Footprint" "Connector_USB:USB_C_Receptacle_Palconn_UTC16-G" (at 162.56 67.31 0)
       (effects (font (size 1.27 1.27)) hide)
     )
